File: pic-rylr998-01/pic-rylr998-01.kicad_pcb (KiCad board)
At the start: 2 copper layers, 28 x 48 mm, 16 parts, among them J1 Conn_02x04_Counter_Clockwise, J2 Conn_01x05_Pin, J3 Screw_Terminal_01x02, U1 LD1117V33

Commit message: cleaned up board silkscreen and made all power supply related tracks 1 mm wide vs default 0.2 mm wide - the three signal lines RA2_LED RA4_PIC_RXD_RYLR998_TXD RA5_PIC_TXD_RYLR998_RXD tracks remain 0.2 mm wide
Parts:
- J1: value Conn_02x04_Counter_Clockwise -> J1
- J2: value Conn_01x05_Pin -> J2
- J3: value Screw_Terminal_01x02 -> J3
Other:
- board size 28 x 48 mm -> 28.5 x 47 mm
